File: audio/audio.kicad_sch (KiCad schematic)
At the start: 4 parts, among them J1 Conn_2Rows-35Pins, U1 TDA7052A

Commit message: add extra ground pins to high speed MIPI LANES for reduction of signal coupling.
Parts:
- J1: footprint (none) -> Connector_Hirose_DF40:Hirose_DF40C-34DP-0.4V_2x17-1MP_P0.4mm
- U1: footprint (none) -> Package_DIP:DIP-8-16_W7.62mm
Changed lines of the file:
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@@
 			)
 		)
-		(property "Footprint" ""
+		(property "Footprint" "Package_DIP:DIP-8-16_W7.62mm"
 			(at 149.86 105.41 0)
 			(effects
@@
 			)
 		)
-		(property "Footprint" ""
+		(property "Footprint" "Connector_Hirose_DF40:Hirose_DF40C-34DP-0.4V_2x17-1MP_P0.4mm"
 			(at 86.36 96.52 0)
 			(effects
