File: display/display_module.kicad_sch (KiCad schematic)
At the start: 0 parts

Commit message: Start work on display module schematic.
Note for later: fix main board PCB, since upon inspection the board has some faults
Parts:
- added C1, C2, C3, C4, C5, C6, C7, C8, C9: 20uF, symbol Device:C_US
- added J1: DISPLAY FPC, symbol Connector_Generic:Conn_2Rows-39Pins
- added J2: FPC LOGIC, symbol Connector_Generic:Conn_01x08
- added J4: DF40, DF40-34P:HIROSE_DF40C-34DS-0.4V_58_, symbol Connector_Generic_MountingPin:Conn_2Rows-35Pins_MountingPin
Connections:
- new net +3.3V: C4.2, C5.2, C6.2, J2.3 (Pin_3), J4.13 (Pin_13)
- new net +3.7VBAT: C7.2, C8.2, C9.2, J4.15 (Pin_15)
- new net +5V: C1.1, C2.1, C3.1, J4.14 (Pin_14)
- new net DSI-0-N: J4.3 (Pin_3)
- new net DSI-0-P: J4.4 (Pin_4)
- new net DSI-1-N: J4.5 (Pin_5)
- new net DSI-1-P: J4.6 (Pin_6)
- new net DSI-2-N: J4.7 (Pin_7)
- new net DSI-2-P: J4.8 (Pin_8)
- new net DSI-3-N: J4.9 (Pin_9)
- new net DSI-3-P: J4.10 (Pin_10)
- new net DSI-CLK-N: J4.1 (Pin_1)
- new net DSI-CLK-P: J4.2 (Pin_2)
- new net GND: C1.2, C2.2, C3.2, C4.1, C5.1, C6.1, C7.1, C8.1, C9.1, J2.1 (Pin_1), J2.8 (Pin_8), J4.16 (Pin_16)
- new net I2C3-SCL: J2.4 (Pin_4), J4.11 (Pin_11)
- new net I2C3-SDA: J2.5 (Pin_5), J4.12 (Pin_12)
- new net RST: J2.7 (Pin_7), J4.17 (Pin_17)

Commit message: finish display module schematic
Parts:
- added R1: 100OHM, symbol Device:R
- J1: footprint (none) -> Connector_FFC-FPC:Amphenol_F32R-1A7x1-11029_1x29-1MP_P0.5mm_Horizontal; symbol Connector_Generic:Conn_2Rows-39Pins -> Connector_Generic:Conn_02x15_Odd_Even
- J2: footprint (none) -> Connector_FFC-FPC:Amphenol_F32Q-1A7x1-11007_1x07-1MP_P0.5mm_Horizontal
Connections:
- net +3.3V: now also J1.27 (Pin_27), J1.28 (Pin_28)
- net +3.7VBAT: now also R1.2
- net DSI-0-N: now also J1.7 (Pin_7)
- net DSI-0-P: now also J1.8 (Pin_8)
- net DSI-1-N: now also J1.10 (Pin_10)
- net DSI-1-P: now also J1.11 (Pin_11)
- net DSI-2-N: now also J1.16 (Pin_16)
- net DSI-2-P: now also J1.17 (Pin_17)
- net DSI-3-N: now also J1.19 (Pin_19)
- net DSI-3-P: now also J1.20 (Pin_20)
- net DSI-CLK-N: now also J1.13 (Pin_13)
- net DSI-CLK-P: now also J1.14 (Pin_14)
- net GND: now also J1.12 (Pin_12), J1.15 (Pin_15), J1.18 (Pin_18), J1.2 (Pin_2), J1.21 (Pin_21), J1.22 (Pin_22), J1.24 (Pin_24), J1.29 (Pin_29), J1.30 (Pin_30), J1.6 (Pin_6), J1.9 (Pin_9)
- net at J1.4 (Pin_4): now also R1.1
Other:
- note added: "D40C Input and Power Smoothing"
- note added: "Display FPC IN"
- note added: "Display FPC LOGIC IN"
- moved on the sheet: C1, C2, C3, C4, C5, C6, C7, C8, C9, J2, J4

Commit message: Finish Display module.
The display module is basically an adapter with no fancy features, I choose to do this so pulsephone is compatible with ALL mipi displays since different manufacturers have different pinouts and standards
Parts:
- C1, C2, C3, C4, C5, C6, C7, C8, C9: footprint (none) -> Capacitor_SMD:C_1206_3216Metric
- J4: footprint DF40-34P:HIROSE_DF40C-34DS-0.4V_58_ -> Connector_Hirose_DF40:Hirose_DF40C(2.0)-70DS-0.4V_2x35_P0.4mm; now not fitted
- R1: value 100OHM -> 100 OHM; footprint (none) -> Resistor_SMD:R_1206_3216Metric
Changed lines of the file:
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@@
 			)
 		)
-		(property "Footprint" ""
+		(property "Footprint" "Capacitor_SMD:C_1206_3216Metric"
 			(at 134.62 55.88 0)
 			(effects
@@
 			)
 		)
-		(property "Footprint" ""
+		(property "Footprint" "Capacitor_SMD:C_1206_3216Metric"
 			(at 55.88 82.55 0)
 			(effects
@@
 			)
 		)
-		(property "Footprint" ""
+		(property "Footprint" "Capacitor_SMD:C_1206_3216Metric"
 			(at 48.26 101.6 0)
 			(effects
@@
 			)
 		)
-		(property "Footprint" ""
+		(property "Footprint" "Capacitor_SMD:C_1206_3216Metric"
 			(at 58.42 101.6 0)
 			(effects
@@
 			)
 		)
-		(property "Footprint" ""
+		(property "Footprint" "Capacitor_SMD:C_1206_3216Metric"
 			(at 66.04 82.55 0)
 			(effects
@@
 			)
 		)
-		(property "Footprint" ""
+		(property "Footprint" "Capacitor_SMD:C_1206_3216Metric"
 			(at 106.68 55.88 0)
 			(effects
@@
 			)
 		)
-		(property "Value" "100OHM"
+		(property "Value" "100 OHM"
 			(at 257.81 70.866 90)
 			(effects
@@
 			)
 		)
-		(property "Footprint" ""
+		(property "Footprint" "Resistor_SMD:R_1206_3216Metric"
 			(at 256.54 75.438 90)
 			(effects
@@
 			)
 		)
-		(property "Footprint" ""
+		(property "Footprint" "Capacitor_SMD:C_1206_3216Metric"
 			(at 120.65 55.88 0)
 			(effects
@@
 			)
 		)
-		(property "Footprint" ""
+		(property "Footprint" "Capacitor_SMD:C_1206_3216Metric"
 			(at 60.96 82.55 0)
 			(effects
@@
 		(in_bom yes)
 		(on_board yes)
-		(dnp no)
+		(dnp yes)
 		(fields_autoplaced yes)
 		(property "Reference" "J4"
@@
 			)
 		)
-		(property "Footprint" "DF40-34P:HIROSE_DF40C-34DS-0.4V_58_"
+		(property "Footprint" "Connector_Hirose_DF40:Hirose_DF40C(2.0)-70DS-0.4V_2x35_P0.4mm"
 			(at 87.63 91.44 0)
 			(effects
@@
 			)
 		)
-		(property "Footprint" ""
+		(property "Footprint" "Capacitor_SMD:C_1206_3216Metric"
 			(at 69.85 101.6 0)
 			(effects

Commit message: final review change (board was ordered, prod ready verSion)
Parts:
- J1: value DISPLAY FPC -> THD THD0515-29CL-SN; footprint Connector_FFC-FPC:Amphenol_F32R-1A7x1-11029_1x29-1MP_P0.5mm_Horizontal -> Connector_FFC-FPC:FPC-29-P0.5
- J2: footprint Connector_FFC-FPC:Amphenol_F32Q-1A7x1-11007_1x07-1MP_P0.5mm_Horizontal -> Connector_FFC-FPC:FPC_7
- J4: footprint Connector_Hirose_DF40:Hirose_DF40C(2.0)-70DS-0.4V_2x35_P0.4mm -> Connector_Hirose_DF40:Hirose_DF40C-34DS-0.4V_2x17_P0.4mm; now fitted
Changed lines of the file:
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@@
 			)
 		)
-		(property "Footprint" "Connector_FFC-FPC:Amphenol_F32Q-1A7x1-11007_1x07-1MP_P0.5mm_Horizontal"
+		(property "Footprint" "Connector_FFC-FPC:FPC_7"
 			(at 110.49 163.83 0)
 			(effects
@@
 			)
 		)
-		(property "Datasheet" "~"
+		(property "Datasheet" ""
 			(at 110.49 163.83 0)
 			(effects
@@
 			)
 		)
-		(property "Description" "Generic connector, single row, 01x08, script generated (kicad-library-utils/schlib/autogen/connector/)"
+		(property "Description" ""
 			(at 110.49 163.83 0)
 			(effects
@@
 		(in_bom yes)
 		(on_board yes)
-		(dnp yes)
+		(dnp no)
 		(fields_autoplaced yes)
 		(property "Reference" "J4"
@@
 			)
 		)
-		(property "Footprint" "Connector_Hirose_DF40:Hirose_DF40C(2.0)-70DS-0.4V_2x35_P0.4mm"
+		(property "Footprint" "Connector_Hirose_DF40:Hirose_DF40C-34DS-0.4V_2x17_P0.4mm"
 			(at 87.63 91.44 0)
 			(effects
@@
 			)
 		)
-		(property "Value" "DISPLAY FPC"
+		(property "Value" "THD THD0515-29CL-SN"
 			(at 237.49 67.31 0)
 			(effects
@@
 			)
 		)
-		(property "Footprint" "Connector_FFC-FPC:Amphenol_F32R-1A7x1-11029_1x29-1MP_P0.5mm_Horizontal"
+		(property "Footprint" "Connector_FFC-FPC:FPC-29-P0.5"
 			(at 236.22 88.9 0)
 			(effects
@@
 			)
 		)
-		(property "Datasheet" "~"
+		(property "Datasheet" ""
 			(at 236.22 88.9 0)
 			(effects
@@
 			)
 		)
-		(property "Description" "Generic connector, double row, 02x15, odd/even pin numbering scheme (row 1 odd numbers, row 2 even numbers), script generated (kicad-library-utils/schlib/autogen/connector/)"
+		(property "Description" ""
 			(at 236.22 88.9 0)
 			(effects
