File: main_board/pulsephone_main_board.kicad_sch (KiCad schematic)
At the start: 93 parts, among them J1 USB_C_Receptacle_USB2.0_14P, J2 Conn_01x05, J3 Conn_2Rows-35Pins_MountingPin, J4 Conn_2Rows-35Pins_MountingPin, J5 Conn_2Rows-35Pins_MountingPin, J6 Conn_01x01_Socket, J7 Micro_SD_Card_Det1, J8 Conn_2Rows-35Pins_MountingPin, U1 AP2112K-3.3, U2 PCM5102APWR, U4 TPS63020DSJR/3.7V Reg, U5 TP4056-42-ESOP8, U6 LBEE5KL1YN-814, Y1 XO53

Commit message: added m.2 connector in place of old wifi.
wifi and bluetooth is now routed to the mainboard with the m.2 connector through SDIO, so no more future wifi module since m.2 feature replaces it.
Parts:
- removed C38: 100nF, Capacitor_SMD:C_0805_2012Metric, symbol Device:C_US
- removed J6: Conn_01x01_Socket, Connector_Coaxial:U.FL_Hirose_U.FL-R-SMT-1_Vertical, symbol Connector:Conn_01x01_Socket
- removed L1: 1µH, Inductor_SMD:L_01005_0402Metric, symbol Device:L
- removed U6: LBEE5KL1YN-814, footprints:XCVR_LBEE5KL1YN-814, symbol LBEE5KL1YN-814:LBEE5KL1YN-814
- removed Y1: XO53, Oscillator:Oscillator_SMD_EuroQuartz_XO53-4Pin_5.0x3.2mm, symbol Oscillator:XO53
- added J9: Bus_M.2_Socket_E, mdt:AMPHENOL_MDT180E03001, symbol Connector:Bus_M.2_Socket_E
Connections:
- net +3.3V: now also J9.2 (3.3V), J9.4 (3.3V), J9.72 (3.3V), J9.74 (3.3V)
- net BT_UART_CTS_N: now also J9.34 (UART_CTS)
- net BT_UART_R: now also J9.22 (UART_RXD)
- net BT_UART_RTS_N: now also J9.36 (UART_RTS)
- net BT_UART_T: now also J9.32 (UART_TXD)
- net GND: now also J9.1 (GND), J9.18 (GND), J9.33 (GND), J9.39 (GND), J9.45 (GND), J9.51 (GND), J9.57 (GND), J9.63 (GND), J9.69 (GND), J9.7 (GND), J9.75 (GND)
- net MOD_GPIO_128: now also J9.56 (~{W_DISABLE1}); no longer J8.22 (Pin_22)
- net MOD_GPIO_130: now also J9.54 (~{W_DISABLE2}); no longer J8.23 (Pin_23)
- net SD2_RST_B: now also J9.23 (~{SDIO_RESET})
- net SDIO_0: now also J9.13 (SDIO_DATA0)
- net SDIO_1: now also J9.15 (SDIO_DATA1)
- net SDIO_2: now also J9.17 (SDIO_DATA2)
- net SDIO_3: now also J9.19 (SDIO_DATA3)
- net SDIO_CLK: now also J9.9 (SDIO_CLK)
- net SDIO_CMD: now also J9.11 (SDIO_CMD)
- net USB_DN: now also MCM93_MOD1.137 (32), J9.5 (USB_D-)
- net USB_DP: now also MCM93_MOD1.136 (31), J9.3 (USB_D+)

Commit message: create new branch
major supply issues with the mcm-imx93, so i am swapping to a new SoM.
Parts:
- removed AUD-L1, AUD-R1: TestPoint, TestPoint:TestPoint_Pad_1.0x1.0mm, symbol Connector:TestPoint
- removed I2C3-SCL1, I2C3-SDA1: TestPoint, TestPoint:TestPoint_Pad_D2.5mm, symbol Connector:TestPoint
- removed MCM93_MOD1: MCM93_MOD, mcm-imx93_footprint:LGA-140-080-30x30-iMX93, symbol mcm-imx93:MCM93_MOD
- added A1, A2, A3: (no value), symbol Connector_SoM:Conn_1x90
Connections:
- net +3.3V: no longer R12.1
- net +5V: now also A3.66, A3.71, A3.73, A3.75, A3.77, A3.79, A3.81, A3.83, A3.85, A3.87, A3.89
- net BT_UART_CTS_N: now also A2.22
- net BT_UART_R: now also A2.20
- net BT_UART_RTS_N: now also A2.26
- net BT_UART_T: now also A2.24
- net CAM_I2C_SCL: now also A1.17
- net CAM_I2C_SDA: now also A1.19
- net CSI_CLK_N: now also A1.89
- net CSI_CLK_P: now also A1.87
- net DSI_CLK_N: now also A3.29
- net DSI_CLK_P: now also A3.31
- net GND: now also R12.1; no longer R12.2, U2.17 (XSMT)
- net I2C3_SCL: now also A2.32
- net I2C3_SDA: now also A2.30
- net MOD_UART6_CTS: no longer J8.8 (Pin_8)
- net MOD_UART6_RTS: no longer J8.7 (Pin_7)
- net MOD_UART6_RX: no longer J8.5 (Pin_5)
- net MOD_UART6_TX: no longer J8.6 (Pin_6)
- net SD2_CD_B: now also A1.74
- net SD2_CLK: now also A1.82
- net SD2_CMD: now also A1.88
- net SD2_DAT0: now also A1.86
- net SD2_DAT1: now also A1.80
- net SD2_DAT2: now also A1.78
- net SD2_DAT3: now also A1.84
- net SD2_RST_B: now also A2.25
- net SD2_VDD: now also A1.90
- net SDIO_0: now also A2.35
- net SDIO_1: now also A2.33
- net SDIO_2: now also A2.31
- net SDIO_3: now also A2.29
- net SDIO_CLK: now also A2.45
- net SDIO_CMD: now also A2.43
- net UART_RX: now also A2.90
- net UART_TX: now also A2.88
- net USB_DN: now also A3.67
- net USB_DP: now also A3.65
- net at U2.6 (OUTL): no longer J5.8 (Pin_8)
- net at U2.7 (OUTR): no longer J5.9 (Pin_9)
- net AUDIO_DATA_OUT renamed AUD_IN
- net AUD_IN: now also A2.70
- net AUDIO_FRAME_CLOCK renamed AUD_FCLK
- net AUD_FCLK: now also A2.64
- net CSI_D0_N renamed CSI_0_N
- net CSI_0_N: now also A1.83
- net CSI_D0_P renamed CSI_0_P
- net CSI_0_P: now also A1.81
- net CSI_D1_N renamed CSI_1_N
- net CSI_1_N: now also A1.75
- net CSI_D1_P renamed CSI_1_P
- net CSI_1_P: now also A1.73
- net DSI_D0_N renamed DSI_0_N
- net DSI_0_N: now also A3.14
- net DSI_D0_P renamed DSI_0_P
- net DSI_0_P: now also A3.12
- net DSI_D1_N renamed DSI_1_N
- net DSI_1_N: now also A3.18
- net DSI_D1_P renamed DSI_1_P
- net DSI_1_P: now also A3.16
- net DSI_D2_N renamed DSI_2_N
- net DSI_2_N: now also A3.25
- net DSI_D2_P renamed DSI_2_P
- net DSI_2_P: now also A3.23
- net DSI_D3_N renamed DSI_3_N
- net DSI_3_N: now also A3.22
- net DSI_D3_P renamed DSI_3_P
- net DSI_3_P: now also A3.20
- net SAI_BITCLOCK renamed SAI_BCK
- net SAI_BCK: now also A2.72
- net SAI_MASTERCLOCK renamed SAI_MCLK
- net SAI_MCLK: now also A2.82
- new net: R12.2, U2.17 (XSMT)
- new net AUD_L: J5.8 (Pin_8)
- new net AUD_R: J5.9 (Pin_9)
- new net MOD_UART_RX: A2.86, J8.5 (Pin_5)
- new net MOD_UART_TX: A2.85, J8.6 (Pin_6)
Other:
- note added: "5V FILTERS"
- note added: "WIFI/BT M.2"
- note removed: "MIPI CSI"
- note removed: "MIPI-DSI"
- note removed: "WIFI/BT"
- moved on the sheet: C14, C15, C16, C17, C18, C19, C2, C20, C21, C22, C23, C24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

Commit message: finish new SoM swapped sch.
Parts:
- removed ON/OFF1: SSSS810701, SSSS810701:SSSS810701, symbol SSSS810701:SSSS810701
- removed R5, R6: 10 kΩ, Resistor_SMD:R_0805_2012Metric, symbol Device:R
- removed RESET1: SW_Push, Button_Switch_SMD:SW_Push_1P1T-SH_NO_CK_KMR2xxG, symbol Switch:SW_Push
- added SW1: SW_Push, symbol Switch:SW_Push
- A1, A2, A3: footprint (none) -> Connector_Hirose_DF40:Hirose_DF40C-90DS-0.4V_2x45_P0.4mm
Connections:
- net MOD_GPIO_115 is gone; now on net GPIO1_IO08: J8.16 (Pin_16)
- net MOD_GPIO_116 is gone; now on net GPIO1_IO10: J8.17 (Pin_17)
- net MOD_GPIO_117 is gone; now on net GPIO1_IO11: J8.18 (Pin_18)
- net MOD_GPIO_118 is gone; now on net GPIO1_IO12: J8.19 (Pin_19)
- net MOD_GPIO_119 is gone; now on net GPIO1_IO14: J8.20 (Pin_20)
- net MOD_GPIO_48 is gone; now on net GPIO1_IO01: J8.12 (Pin_12)
- net MOD_GPIO_95 is gone; now on net GPIO1_IO03: J8.13 (Pin_13)
- net MOD_GPIO_96 is gone; now on net GPIO1_IO05: J8.14 (Pin_14)
- net MOD_GPIO_99 is gone; now on net GPIO1_IO06: J8.15 (Pin_15)
- net MOD_I2C7_SCL is gone; now on net GND: J8.9 (Pin_9)
- net MOD_I2C8_SDA is gone; now on net GND: J8.10 (Pin_10)
- net GND: now also SW1.1
- net ONOFF: now also SW1.2
- net GPIO1_IO11: now reaches A3.30
- net GPIO1_IO14: now reaches A3.48
- net GPIO1_IO12: now reaches A3.50
- net GPIO1_IO10: now reaches A3.52
- net GPIO1_IO03: now reaches A3.54
- net GPIO1_IO06: now reaches A3.58
- net GPIO1_IO08: now reaches A3.60
- net GPIO1_IO05: now reaches A3.62
- net GPIO1_IO01: now reaches A3.64
- net MOD_GPIO_120: no longer names the net of J8.21 (Pin_21)
- net MOD_I2C8_SCL: no longer names the net of J8.11 (Pin_11)
Other:
- note added: "ON/OFF"
- note removed: "Active Low ONOFF"
- note removed: "Active Low Reset"
- moved on the sheet: C14, C15, C16, C17, C18, C19, C20, C21, C22, C23, C24, C25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
