File: main_board/_restore_backup_2026-09-20T22-07-57-618/pulsephone_main_board.kicad_sch (KiCad schematic)
At the start: 85 parts, among them J1 USB_C_Receptacle_USB2.0_14P, J2 Conn_01x05, J3 Conn_2Rows-35Pins_MountingPin, J4 Conn_2Rows-35Pins_MountingPin, J5 Conn_2Rows-35Pins_MountingPin, J7 Micro_SD_Card_Det1, J8 Conn_2Rows-35Pins_MountingPin, J9 Bus_M.2_Socket_E, SW1 SW_Push, U1 AP2112K-3.3, U2 PCM5102APWR, U4 TPS63020DSJR/3.7V Reg, U5 TP4056-42-ESOP8

Commit message: test
Parts:
- removed R5: 10kOHM, Resistor_SMD:R_0603_1608Metric_Pad0.98x0.95mm_HandSolder, symbol Device:R
- A1, A2, A3: KiLib_Generator connector/generator -> (none)
- D7, D8, F1, F2, R12, R13: KiLib_Generator SMD_2terminal_chip_molded -> (none)
- SW1: footprint EVQ-P7A01P:SW_EVQ-P7A01P -> (none)
Connections:
- net +3.3V: no longer J7.4 (VDD)
- net +3.7VBAT: now also U3.6 (EN)
- net +5V: now also A3.66
- net AUD_L: no longer U2.6 (OUTL)
- net AUD_R: no longer U2.7 (OUTR)
- net GND: no longer A1.18, A1.21, A1.30, A1.33, A1.49, A1.76, A1.85, A2.18, A2.23, A2.47, A2.53, A2.75, A2.84, A3.10, A3.15, A3.21, A3.24, A3.27, A3.33, A3.34, A3.39, A3.45, A3.51, A3.57, A3.63, A3.68, A3.74, A3.9
- net MOD_GPIO_128: no longer A3.40
- net MOD_GPIO_130: no longer A3.38
- net ONOFF: no longer A1.20
- net SD2_VDD: now reaches A1.90
- net SD2_VDD: now also J7.4 (VDD)
- net VBUS: no longer names the net of C12.2, J1.A4 (VBUS), J1.A9 (VBUS), J1.B4 (VBUS), J1.B9 (VBUS), U5.4 (V_{CC}), U5.8 (CE)
- net VBUS: no longer A3.66
